File: plc/kicad/LibrePLC32.kicad_pcb (KiCad board)
At the start: 4 copper layers, 279 parts, among them CN1 DB128V-5.08-2P-GN-S, CN10 DB128V-5.08-2P-GN-S, CN11 DB2ERC-5.08-4P, CN12 DB2ERC-5.08-4P, CN13 DB128V-5.08-2P-GN-S, CN14 DB128V-5.08-2P-GN-S, CN2 DB128V-5.08-2P-GN-S, CN3 DB128V-5.08-2P-GN-S, CN4 DB128V-5.08-2P-GN-S, CN5 DB128V-5.08-2P-GN-S, CN6 DB128V-5.08-2P-GN-S, CN7 DB128V-5.08-2P-GN-S, CN8 DB128V-5.08-2P-GN-S, CN9 DB128V-5.08-2P-GN-S, J2 Conn_01x04_Pin, J3 Conn_01x02_Pin, Q1 AO3400A, Q2 AO3400A, Q3 L8050QLT1G, Q4 L8050QLT1G, Q5 BSS138LT1G, Q6 CSD19537Q3, SW1 TSD003B08026A03, SW2 TSD003B08026A03, SW3 TSD003B08026A03, SW4 MSK12C02, SW5 MSK12C02, U1 TCA9535PWR, U10 ESP32-S3-MINI-1U, U11 BS-0601-SK-4W, U12 AHT20_C2757850, U13 CP2102N-A02-GQFN28R, U14 LMR16006XDDCR, U15 TPS54560BDDAR, U16 TPS26630RGER, U17 TPS7A5201QRGRRQ1, U18 TCAN337DR, U19 THVD1450DR, U2 TPS272C45DRHFR, U20 W5500, U3 TPS272C45DRHFR, U4 ADS1115IDGSR, U5 LTV-814S-TA1-A, U6 LTV-814S-TA1-A, U7 LTV-814S-TA1-A, U8 LTV-814S-TA1-A, U9 RV-3028-C7, X1 X322525MRB4SI

Commit message: Updated PCB placement
Parts:
- moved C12 417.2 mm to (-141.2, 155.1)
- moved C13 417.2 mm to (-141.2, 158.6)
- moved U11 417.2 mm to (-138.7, 144.8)
- moved R44 417.2 mm to (-135.5, 158.1)
- moved U9 417.2 mm to (-138.5, 157.1)
- moved C15 403.0 mm to (-182.9, 188.9)
- moved U12 403.0 mm to (-186.3, 188.8)
- moved TP27 370.5 mm to (-170.4, 234.8), turned to 90 degrees
- moved TP28 338.5 mm to (-138.9, 235.1), turned to 90 degrees
- moved TP32 326.0 mm to (-120.6, 201.8)
- moved TP31 320.9 mm to (-115.1, 197.9)
- moved D3 277.5 mm to (-223.3, 225.4)
- moved D4 277.5 mm to (-223.3, 221.0)
- moved R49 277.5 mm to (-220.0, 225.4)
- moved R50 277.5 mm to (-219.9, 221.1)
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Connections:
- C10 pad 1: /Terminal Blocks Interface/MCU_DI4 -> /MCU/MCU_DI4
- C7 pad 1: /Terminal Blocks Interface/MCU_DI1 -> /MCU/MCU_DI1
- C8 pad 1: /Terminal Blocks Interface/MCU_DI2 -> /MCU/MCU_DI2
- C9 pad 1: /Terminal Blocks Interface/MCU_DI3 -> /MCU/MCU_DI3
- R36 pad 1: /Terminal Blocks Interface/MCU_DI1 -> /MCU/MCU_DI1
- R37 pad 1: /Terminal Blocks Interface/MCU_DI2 -> /MCU/MCU_DI2
- R38 pad 1: /Terminal Blocks Interface/MCU_DI3 -> /MCU/MCU_DI3
- R39 pad 1: /Terminal Blocks Interface/MCU_DI4 -> /MCU/MCU_DI4
Routing:
- net +3V3: track 170.8 -> 139.4 mm
- net GND: track 279.3 -> 301.3 mm
- net /Power/V_IN_MAIN: track 58.0 -> 73.2 mm
- net V_FIELD: track 20.6 -> 24.8 mm
- net /Terminal Blocks Interface/MCU_DI3: track 3.36 -> 0.00 mm
- net /MCU/MCU_DI3: track 0.00 -> 3.36 mm
- net /MCU/MCU_DI4: track 0.00 -> 3.13 mm
- net /Terminal Blocks Interface/MCU_DI1: track 3.13 -> 0.00 mm
- net /MCU/MCU_DI2: track 0.00 -> 3.13 mm
- net /MCU/MCU_DI1: track 0.00 -> 3.13 mm
- net /Terminal Blocks Interface/MCU_DI4: track 3.13 -> 0.00 mm
- net /Terminal Blocks Interface/MCU_DI2: track 3.13 -> 0.00 mm
- net /Terminal Blocks Interface/DI1: track 9.38 -> 10.7 mm
- net /Terminal Blocks Interface/DI2: track 9.38 -> 10.1 mm
- net /MCU/I2C_SCL: track 27.7 -> 27.2 mm

Commit message: Added mounting holes & PCB outline
Parts:
- added H1: MountingHole_Pad, MountingHole:MountingHole_4.3mm_M4_DIN965_Pad_TopBottom, F.Cu at (57.3, 146.2)
- added H2: MountingHole_Pad, MountingHole:MountingHole_4.3mm_M4_DIN965_Pad_TopBottom, F.Cu at (199.9, 146.3)
- added H3: MountingHole_Pad, MountingHole:MountingHole_4.3mm_M4_DIN965_Pad_TopBottom, F.Cu at (170.4, 43.7)
- added H4: MountingHole_Pad, MountingHole:MountingHole_4.3mm_M4_DIN965_Pad_TopBottom, F.Cu at (81.0, 43.7)
- moved C11 304.1 mm to (127.7, 43.6)
- moved R45 304.1 mm to (124.7, 43.6)
- moved SW1 304.1 mm to (126.9, 50.6)
- moved CN6 298.1 mm to (107.1, 146.2)
- moved CN7 298.1 mm to (96.8, 146.2)
- moved CN8 298.1 mm to (86.6, 146.2)
- moved CN2 298.0 mm to (127.5, 146.2)
- moved CN9 298.0 mm to (76.4, 146.2)
- moved CN1 298.0 mm to (117.2, 146.2)
- moved C19 297.8 mm to (143.7, 103.0)
- moved C2 297.8 mm to (142.9, 129.2)
- moved C26 297.8 mm to (114.4, 99.8)
- moved C3 297.8 mm to (145.5, 128.4)
- moved C33 297.8 mm to (135.6, 80.2)
- moved C36 297.8 mm to (139.2, 80.2)
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Connections:
- D1 pad 1: ++5V -> +5V
- D12 pad 1: ++5V -> +5V
- D13 pad 1: ++5V -> +5V
- D2 pad 1: ++5V -> +5V
- RLY1 pad 4: ++5V -> +5V
- RLY2 pad 4: ++5V -> +5V
Routing:
- net V_FIELD: track 24.8 -> 160.0 mm, vias 67 -> 79
- net /CAN/CAN_TX: track 0.00 -> 92.8 mm, vias 0 -> 2
- net /CAN/CAN_RX: track 0.00 -> 85.7 mm, vias 0 -> 2
- net /RS-485/RS485_RXD: track 8.74 -> 88.0 mm
- net /RS-485/RS485_DIR: track 10.6 -> 88.0 mm
- net /RS-485/RS485_TXD: track 7.26 -> 83.7 mm
- net /MCU/I2C_SDA: track 25.5 -> 68.7 mm, vias 2 -> 4
- net /MCU/I2C_SCL: track 27.2 -> 67.0 mm, vias 2 -> 4
- net GND: track 301.3 -> 340.7 mm, vias 296 -> 293
- net /Terminal Blocks Interface/DI_COM: track 44.3 -> 81.6 mm
- net PWR_RS485: track 3.62 -> 18.1 mm
- net +5V: track 52.8 -> 67.2 mm
- net ++5V: track 14.4 -> 0.00 mm
- net PWR_CAN: track 3.72 -> 10.1 mm
- net /MCU/~{MCU_RST}: track 14.6 -> 18.6 mm
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- added copper zone on In1.Cu, net GND
- added copper zone on In2.Cu, net GND
Other:
- board outline added: 154.5 x 112.9 mm
