File: plc/kicad/LibrePLC32.kicad_sch (KiCad schematic)
At the start: 0 parts

Commit message: Added setup leds & shared SPI bus
Other:
- sheet Ethernet ports: added SPI_MISO, SPI_MOSI, SPI_SCLK; removed ETH_MISO, ETH_MOSI, ETH_SCLK
- sheet MCU ports: added SPI_MISO, SPI_MOSI, SPI_SCLK; removed ETH_MISO, ETH_MOSI, ETH_SCLK
Changed lines of the file:
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@@
 			)
 		)
-		(pin "ETH_SCLK" output
+		(pin "SPI_SCLK" output
 			(at 127 134.62 180)
 			(effects
@@
 			)
 		)
-		(pin "ETH_MOSI" output
+		(pin "SPI_MOSI" output
 			(at 127 129.54 180)
 			(effects
@@
 			)
 		)
-		(pin "ETH_MISO" input
+		(pin "SPI_MISO" input
 			(at 127 132.08 180)
 			(effects
@@
 			)
 		)
-		(pin "ETH_MOSI" input
+		(pin "SPI_MOSI" input
 			(at 82.55 129.54 0)
 			(effects
@@
 			)
 		)
-		(pin "ETH_MISO" output
+		(pin "SPI_MISO" output
 			(at 82.55 132.08 0)
 			(effects
@@
 			)
 		)
-		(pin "ETH_SCLK" input
+		(pin "SPI_SCLK" input
 			(at 82.55 134.62 0)
 			(effects

Commit message: Changed CAN & RS485 to input voltage unprotected
Other:
- sheet Power ports: added V_IN_UNPROTECTED; removed none
- sheet Terminal Blocks Interface ports: added V_IN_UNPROTECTED; removed none
Changed lines of the file:
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@@
+	(wire
+		(pts
+			(xy 207.01 53.975) (xy 207.01 82.55)
+		)
+		(stroke
+			(width 0)
+			(type default)
+		)
+	)
 	(wire
 		(pts
@@
 		)
 	)
+	(wire
+		(pts
+			(xy 207.01 82.55) (xy 218.44 82.55)
+		)
+		(stroke
+			(width 0)
+			(type default)
+		)
+	)
 	(polyline
 		(pts
@@
 		(pts
 			(xy 82.55 140.97) (xy 127 140.97)
+		)
+		(stroke
+			(width 0)
+			(type default)
+		)
+	)
+	(wire
+		(pts
+			(xy 218.44 53.975) (xy 207.01 53.975)
 		)
 		(stroke
@@
 			)
 		)
+		(pin "V_IN_UNPROTECTED" output
+			(at 218.44 82.55 180)
+			(effects
+				(font
+					(size 1.27 1.27)
+				)
+				(justify left)
+			)
+		)
 		(instances
 			(project "LibrePLC32"
@@
 			(effects
 				(font
+					(size 1.27 1.27)
+				)
+				(justify left)
+			)
+		)
+		(pin "V_IN_UNPROTECTED" input
+			(at 218.44 53.975 180)
+			(effects
+				(font

Commit message: Added isolated CAN bus
Other:
- sheet CAN ports: added none; removed CAN_FAULT
- sheet MCU ports: added none; removed CAN_FAULT
Changed lines of the file:
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@@
-	(wire
-		(pts
-			(xy 82.55 84.455) (xy 127 84.455)
-		)
-		(stroke
-			(width 0)
-			(type default)
-		)
-	)
 	(wire
 		(pts
@@
 			)
 		)
-		(pin "CAN_FAULT" output
-			(at 82.55 84.455 0)
-			(effects
-				(font
-					(size 1.27 1.27)
-				)
-				(justify right)
-			)
-		)
 		(pin "CAN_RX" output
 			(at 82.55 79.375 0)
@@
 			(effects
 				(font
-					(size 1.27 1.27)
-				)
-				(justify left)
-			)
-		)
-		(pin "CAN_FAULT" input
-			(at 127 84.455 180)
-			(effects
-				(font

Commit message: Added more mounting holes
Parts:
- added H1, H2, H3, H4, H5, H6, H7, H8: MountingHole_Pad, MountingHole:MountingHole_4.3mm_M4_DIN965_Pad_TopBottom, symbol Mechanical:MountingHole_Pad
Connections:
- new net GND: H1.1, H2.1, H3.1, H4.1, H5.1, H6.1, H7.1, H8.1
