File: plc/kicad/LibrePLC32.kicad_sch (KiCad schematic)
At the start: 8 parts

Commit message: Add schematic digital output expansion
Co-authored-by: arena-agent <297053741+arena-agent@users.noreply.github.com>
Other:
- added sheet Digital Output Expansion (output_expansion.kicad_sch)
Changed lines of the file:
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@@
 		)
+	)
+	(sheet
+		(at 127 164)
+		(size 57.15 22.86)
+		(exclude_from_sim no)
+		(in_bom yes)
+		(on_board no)
+		(dnp no)
+		(fields_autoplaced yes)
+		(stroke (width 0.1524) (type solid))
+		(fill (color 0 0 0 0))
+		(property "Sheetname" "Digital Output Expansion"
+			(at 127 163.2884 0) (show_name no) (do_not_autoplace no)
+			(effects (font (size 1.27 1.27)) (justify left bottom))
+		)
+		(property "Sheetfile" "output_expansion.kicad_sch"
+			(at 127 187.5716 0) (show_name no) (do_not_autoplace no)
+			(effects (font (size 1.27 1.27)) (justify left top))
+		)
+		(instances (project "LibrePLC32" (path "/ef4c1a27-85a3-413a-9f93-a41c4f97eee5" (page "9"))) )
 	)
 	(sheet_instances
